Commit message: [add] support sim-urdf-schema

File: colcon_ws/src/diffbot_description/robots/diffbot.urdf.xacro (robot description, xacro)
@@ -8,8 +8,10 @@
   <xacro:include filename="$(find diffbot_description)/ros2_control/diffbot.ros2_control.xacro" />
   <!-- Import diffbot isaac description -->
-  <xacro:include filename="$(find diffbot_description)/unity/diffbot.unity.xacro" />
+  <xacro:include filename="$(find diffbot_description)/gazebo/diffbot.gazebo.xacro" />
+  <xacro:include filename="$(find diffbot_description)/unity/diffbot.simulation.xacro" />
   <xacro:diffbot prefix="$(arg prefix)" use_sim="$(arg use_sim)"/>
   <xacro:diffbot_ros2_control
     name="diffbot" prefix="$(arg prefix)" use_sim="$(arg use_sim)" />
-  <xacro:diffbot_unity prefix="$(arg prefix)"/>
+  <xacro:diffbot_gazebo prefix="$(arg prefix)"/>
+  <xacro:diffbot_simulation prefix="$(arg prefix)"/>
 </robot>

File: colcon_ws/src/diffbot_description/robots/diffbot_description.urdf.xacro (robot description, xacro)
@@ -11,10 +11,10 @@
     <color rgba="1.0 1.0 1.0 1.0"/>
   </material>
-  <physics_material name="wheel">
+  <collision_material name="wheel">
     <friction static="1.0" dynamic="1.0"/>
-  </physics_material>
-  <physics_material name="ball">
+  </collision_material>
+  <collision_material name="ball">
     <friction static="0.0" dynamic="0.0"/>
-  </physics_material>
+  </collision_material>
   <xacro:macro name="wheel_macro" params="parent prefix xyz">
     <joint name="${prefix}_joint" type="continuous">
@@ -23,5 +23,6 @@
       <child  link="${prefix}_link"/>
       <origin xyz="${xyz}" rpy="${radians(-90)} 0 0"/>
-      <unity_drive_api stiffness="0" damping="30000" force_limit="1000000"/>
+      <stiffness>0.0</stiffness>
+      <damping>30000.0</damping>
     </joint>
     <link name="${prefix}_link">
@@ -41,5 +42,5 @@
           <cylinder radius="0.05" length="0.02" />
         </geometry>
-        <physics_material name="wheel"/>
+        <collision_material name="wheel"/>
       </collision>
     </link>
@@ -97,5 +98,5 @@
         <sphere radius="0.02" />
       </geometry>
-      <physics_material name="ball"/>
+      <collision_material name="ball"/>
     </collision>
     <inertial>

File: colcon_ws/src/diffbot_description/simulation/diffbot.simulation.xacro (robot description, xacro)
@@ -1,9 +1,9 @@
 <?xml version="1.0"?>
 <robot xmlns:xacro="http://ros.org/wiki/xacro">
-  <xacro:macro name="diffbot_unity" params="prefix">
-    <!-- =============== Isaac Sim =============== -->
-    <unity>
+  <xacro:macro name="diffbot_simulation" params="prefix">
+    <!-- =============== Simulation =============== -->
+    <simulation>
       <sensor name="lidar_link" type="lidar">
-        <update_rate>10</update_rate>
+        <update_rate>30</update_rate>
         <ray>
           <scan>
@@ -30,5 +30,5 @@
       </sensor>
       <sensor name="camera_link" type="camera">
-        <update_rate>30.0</update_rate>
+        <update_rate>10.0</update_rate>
         <horizontal_fov>1.3962634</horizontal_fov>
         <image>
@@ -61,5 +61,5 @@
         <frameName>depth_camera_link</frameName>
       </sensor>
-    </unity>
+    </simulation>
   </xacro:macro>
 </robot>
