Commit message: [add] diffbot に磁気誘導センサと GNSS アンテナを載せる
新しいセンサを試すのに、まずロボット側に載っていないと始まらない。

磁気誘導センサのバーは車体の前、床から 30 mm (base_link で x=0.12, z=0.03)。
実機の MGS1600 / UDS-1213 の取り付け高さに合わせてある。リンクに collision を
付けていないのは、自分が下へ打つレイを自分で遮ってしまうため。

GNSS アンテナはマスト上 (base_link で z=0.35)。衛星の見え方はアンテナの高さと
位置で決まるので、車体自身の影に入らない高さに出す。gnss と gnss_sky_view の
2 つを同じリンクに宣言する: 前者が受信機モデル、後者がその入力になる空の
レイトレースで、後者は ROS へは何も publish しない。

どちらも use_magnetic_guide / use_gnss で外せる。反射 (NLOS) の探索は既定の
2.5 度間隔で 1 回あたり 3000 本ほどレイを打つので、要らない環境では切れた方が
よい。

Co-Authored-By: Claude Opus 5 (1M context) <noreply@anthropic.com>

File: colcon_ws/src/diffbot_description/robots/diffbot.urdf.xacro (robot description, xacro)
@@ -4,4 +4,7 @@
   <xacro:arg name="prefix" default="" />
   <xacro:arg name="use_sim" default="false" />
+  <!-- v1.4.0 の新センサ。1 フレームあたりの計算を増やしたくないときは false -->
+  <xacro:arg name="use_magnetic_guide" default="true" />
+  <xacro:arg name="use_gnss" default="true" />
   <xacro:include filename="$(find diffbot_description)/robots/diffbot_description.urdf.xacro" />
   <!-- Import diffbot ros2_control description -->
@@ -10,8 +13,10 @@
   <xacro:include filename="$(find diffbot_description)/gazebo/diffbot.gazebo.xacro" />
   <xacro:include filename="$(find diffbot_description)/simulation/diffbot.simulation.xacro" />
-  <xacro:diffbot prefix="$(arg prefix)" use_sim="$(arg use_sim)"/>
+  <xacro:diffbot prefix="$(arg prefix)" use_sim="$(arg use_sim)"
+    use_magnetic_guide="$(arg use_magnetic_guide)" use_gnss="$(arg use_gnss)"/>
   <xacro:diffbot_ros2_control
     name="diffbot" prefix="$(arg prefix)" use_sim="$(arg use_sim)" />
   <xacro:diffbot_gazebo prefix="$(arg prefix)"/>
-  <xacro:diffbot_simulation prefix="$(arg prefix)"/>
+  <xacro:diffbot_simulation prefix="$(arg prefix)"
+    use_magnetic_guide="$(arg use_magnetic_guide)" use_gnss="$(arg use_gnss)"/>
 </robot>

File: colcon_ws/src/diffbot_description/robots/diffbot_description.urdf.xacro (robot description, xacro)
@@ -1,5 +1,5 @@
 <?xml version="1.0"?>
 <robot xmlns:xacro="http://ros.org/wiki/xacro">
-  <xacro:macro name="diffbot" params="prefix use_sim:=^|false">
+  <xacro:macro name="diffbot" params="prefix use_sim:=^|false use_magnetic_guide:=^|true use_gnss:=^|true">
   <material name="gray">
     <color rgba="0.5 0.5 0.5 0.2"/>
@@ -211,4 +211,38 @@
     -->
   </link>
+  <!-- 磁気誘導センサのバー。リンク原点がバー面の中心で、+x 前方 / +y 左 /
+       -z が見ている向き。実機と同じく床から 30 mm の高さに置く
+       (base_link から x=0.12, z=0.03)。collision を付けると自分のレイを
+       遮ってしまうので、ジオメトリは持たせない。 -->
+  <xacro:if value="${use_magnetic_guide}">
+  <joint name="magnetic_guide_joint" type="fixed">
+    <parent link="body_link"/>
+    <child  link="magnetic_guide_link"/>
+    <origin xyz="0.19 0 -0.04" rpy="0 0 0"/>
+  </joint>
+  <link name="magnetic_guide_link">
+    <inertial>
+      <origin xyz="0 0 0" rpy="0 0 0"/>
+      <mass value="0.05"/>
+      <inertia ixx="0.0001" ixy="0.0" ixz="0.0" iyy="0.0001" iyz="0.0" izz="0.0001"/>
+    </inertial>
+  </link>
+  </xacro:if>
+  <!-- GNSS アンテナ。衛星の見え方はアンテナの高さと位置で決まるので、
+       車体自身の影に入らないようマスト上 (base_link から z=0.35) に置く。 -->
+  <xacro:if value="${use_gnss}">
+  <joint name="gnss_antenna_joint" type="fixed">
+    <parent link="body_link"/>
+    <child  link="gnss_antenna_link"/>
+    <origin xyz="0 0 0.28" rpy="0 0 0"/>
+  </joint>
+  <link name="gnss_antenna_link">
+    <inertial>
+      <origin xyz="0 0 0" rpy="0 0 0"/>
+      <mass value="0.05"/>
+      <inertia ixx="0.0001" ixy="0.0" ixz="0.0" iyy="0.0001" iyz="0.0" izz="0.0001"/>
+    </inertial>
+  </link>
+  </xacro:if>
   </xacro:macro>
 </robot>

File: colcon_ws/src/diffbot_description/simulation/diffbot.simulation.xacro (robot description, xacro)
@@ -1,5 +1,5 @@
 <?xml version="1.0"?>
 <robot xmlns:xacro="http://ros.org/wiki/xacro">
-  <xacro:macro name="diffbot_simulation" params="prefix">
+  <xacro:macro name="diffbot_simulation" params="prefix use_magnetic_guide:=^|true use_gnss:=^|true">
     <!-- =============== Simulation =============== -->
     <simulation>
@@ -61,4 +61,58 @@
         <frameName>depth_camera_link</frameName>
       </sensor>
+      <!-- ============ v1.4.0: 磁気誘導 (ラインセンサ) ============ -->
+      <!-- AGV 用の磁気ラインセンサ (MGS1600 / UDS-1213 相当)。バー幅 160 mm を
+           1 mm ピッチの素子で見て、テープの横位置 [m] (+左) と左右マーカを
+           simulation_extra_interfaces/MagneticGuide で
+           /diffbot/magnetic_guide_link/magnetic_guide に publish する。
+           テープは sim_props_description の magnetic_course を spawn して置く。
+           min/max_height はバー面 (床上 30 mm) からの測定可能距離。 -->
+      <xacro:if value="${use_magnetic_guide}">
+      <sensor name="magnetic_guide_link" type="magnetic_guide">
+        <update_rate>50</update_rate>
+        <width>0.16</width>
+        <pitch>0.001</pitch>
+        <min_height>0.01</min_height>
+        <max_height>0.06</max_height>
+        <fork>nearest</fork>
+        <noise>
+          <stddev>0.0</stddev>
+        </noise>
+      </sensor>
+      </xacro:if>
+      <!-- ============ v1.4.0: GNSS (受信機モデル + 空の見え方) ============ -->
+      <!-- gnss_sky_view がアンテナから衛星ごとにレイを打ち、直達 / 反射 (NLOS) /
+           遮蔽を判定する。これ自体は ROS へ publish せず、同じリンクの
+           <sensor type="gnss"> が受信機モデルの入力として読む。gnss_canyon を
+           spawn してビルの谷間に入れると測位品質が落ちる様子が見られる。
+           gnss_sky_view が無いときは受信機は真値をそのまま報告する。
+           stochastic_error を false にすると乱数由来の誤差が消え、幾何が生む
+           誤差だけが残るので、同じ場所では毎回同じ誤差になる。 -->
+      <xacro:if value="${use_gnss}">
+      <sensor name="gnss_antenna_link" type="gnss">
+        <update_rate>5.0</update_rate>
+        <origin_latitude>36.549774</origin_latitude>
+        <origin_longitude>139.928772</origin_longitude>
+        <origin_altitude>100.0</origin_altitude>
+        <reconvergence_sec>8.0</reconvergence_sec>
+        <lock_seconds_for_fix>8.0</lock_seconds_for_fix>
+        <wrong_fix_probability>0.01</wrong_fix_probability>
+        <stochastic_error>true</stochastic_error>
+        <seed>20260914</seed>
+      </sensor>
+      <sensor name="gnss_antenna_link" type="gnss_sky_view">
+        <update_rate>5.0</update_rate>
+        <satellite_count>24</satellite_count>
+        <elevation_mask>15.0</elevation_mask>
+        <max_range>500.0</max_range>
+        <seed>1</seed>
+        <!-- 雑草や磁気テープはトリガコライダなので、既定 (false) のままなら衛星を遮らない -->
+        <hit_triggers>false</hit_triggers>
+        <!-- 1 バウンス反射 (NLOS) の探索。spacing を半分にするとレイ数は 4 倍 -->
+        <reflections>true</reflections>
+        <reflection_spacing>2.5</reflection_spacing>
+        <reflection_loss_db>-13.0</reflection_loss_db>
+      </sensor>
+      </xacro:if>
     </simulation>
   </xacro:macro>
