Commit message: [update] diffbot URDF

File: colcon_ws/src/diffbot_description/robots/diffbot_description.urdf.xacro (robot description, xacro)
@@ -13,8 +13,36 @@
   <collision_material name="wheel">
     <friction static="1.0" dynamic="1.0"/>
+    <contact_offset value="0.02"/>
   </collision_material>
   <collision_material name="ball">
     <friction static="0.0" dynamic="0.0"/>
   </collision_material>
+  <!-- buoyancy_material の定義（robot直下） -->
+  <buoyancy_material name="light_material">
+    <density value="0.5"/>  <!-- 水より軽い -->
+  </buoyancy_material>
+  <buoyancy_material name="heavy_material">
+    <density value="2.0"/>  <!-- 水より重い -->
+  </buoyancy_material>
+  <!-- ロボット全体のデフォルト水力学パラメータ（オプション） -->
+  <hydrodynamics>
+    <water_density>1027</water_density>
+    <velocity_reference>1.0</velocity_reference>
+    <pressure_drag>
+      <C_PD1>10</C_PD1>
+      <C_PD2>10</C_PD2>
+      <f_P>0.5</f_P>
+    </pressure_drag>
+    <suction_drag>
+      <C_SD1>10</C_SD1>
+      <C_SD2>10</C_SD2>
+      <f_S>0.5</f_S>
+    </suction_drag>
+    <slamming>
+      <power>2</power>
+      <max_acceleration>10</max_acceleration>
+      <multiplier>1</multiplier>
+    </slamming>
+  </hydrodynamics>
   <xacro:macro name="wheel_macro" params="parent prefix xyz">
     <joint name="${prefix}_joint" type="continuous">
@@ -23,6 +51,6 @@
       <child  link="${prefix}_link"/>
       <origin xyz="${xyz}" rpy="${radians(-90)} 0 0"/>
-      <stiffness>0.0</stiffness>
-      <damping>30000.0</damping>
+      <drive stiffness="0.0" damping="30000.0"/>
+      <limit effort="100.0" velocity="100.0"/>
     </joint>
     <link name="${prefix}_link">
@@ -39,4 +67,5 @@
       </visual>
       <collision>
+        <buoyancy_material name="light_material"/>
         <geometry>
           <cylinder radius="0.05" length="0.02" />
@@ -73,4 +102,13 @@
     <collision>
       <origin xyz="0 0 0" rpy="0 0 0" />
+      <buoyancy_material name="light_material"/>
+      <!-- 水力学パラメータ（リンク固有値を設定）-->
+      <hydrodynamics>
+        <pressure_drag>
+          <C_PD1>15</C_PD1>
+          <C_PD2>20</C_PD2>
+          <f_P>0.5</f_P>
+        </pressure_drag>
+      </hydrodynamics>
       <geometry>
         <box size="0.24 0.178 0.06" />
@@ -95,4 +133,5 @@
     <collision>
       <origin xyz="0 0 0" rpy="0 0 0" />
+      <buoyancy_material name="light_material"/>
       <geometry>
         <sphere radius="0.02" />
