Commit message: [fix] 実機環境で通した結果を反映する
シミュレータ v1.4.0 を Docker で動かして 3 機能を一通り確認した。その場で
分かった食い違いを直す。

gnss_canyon は幅 8 m・高さ 10 m では足りなかった。使用衛星が 20 → 11 に減り
HDOP も 0.60 → 1.18 に上がるものの、RTK Fix は保たれたまま。街路軸の方向の空は
塞げないので、幅 4 m・高さ 12 m まで狭めて初めて Float や単独測位まで落ちる。
README には実測した等級のラダーを載せた。書いてあることと動くものが違うのが
一番たちが悪いので、数字はその場で取ったものにしてある。

前提条件から Unity を外した。イメージがリリース済みの Linux ビルドを落として
コンテナ内で実行するので、このリポジトリを使うのに Unity は要らない。要るのは
シミュレータをソースからビルドするときだけで、それは別リポジトリの話。

追従ノードのゲインは既定のまま。コースは回れるが詰めた値ではないので、
パラメータであることを README に書き足すにとどめた。

Co-Authored-By: Claude Opus 5 (1M context) <noreply@anthropic.com>

File: colcon_ws/src/sim_props_description/urdf/gnss_canyon.urdf (robot description, URDF)
Before this commit: robot gnss_canyon, 2 links, 1 joints
Links:
- link buildings_link: geometry collision box size=6.0 0.6 12.0; collision box size=6.0 0.6 12.0
